File: EL_Electrical/Autre/Accumulator indicator voltage/Indicator_voltage_TNN_V1.0.brd (EAGLE design)
At the start: 74.9 x 55.9 mm, 55 parts, among them J2 22-27-2021

Commit message: Finalisation_carte_élec_V1.0
Parts:
- R10: value 10kΩ, 2W -> 100Ω
- moved R10 1.27 mm to (35.6, 26.7), turned to 0 degrees
Connections:
- new net N$33: NMOS.1, R10.1
- net N$22: now also R10.2; no longer NMOS.1, R10.1
- net V-: no longer R10.2
Routing:
- net N$33: track 0.00 -> 8.32 mm
- net N$22: track 19.6 -> 14.3 mm, vias 2 -> 0
Changed lines of the file:
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@@
 <wire x1="80.01" y1="13.97" x2="80.01" y2="69.85" width="0.0762" layer="20"/>
 <wire x1="80.01" y1="69.85" x2="5.08" y2="69.85" width="0.0762" layer="20"/>
+<text x="10.541" y="65.151" size="3.81" layer="25">TS</text>
 </plain>
 <attributes>
@@
 <attribute name="VALUE" x="12.7" y="15.84" size="0.6096" layer="27"/>
 </element>
-<element name="R10" library="rcl" library_urn="urn:adsk.eagle:library:334" package="R0603" package3d_urn="urn:adsk.eagle:package:23555/3" value="10kΩ, 2W" x="35.56" y="27.94" smashed="yes" rot="R270">
-<attribute name="NAME" x="34.925" y="27.305" size="0.6096" layer="25" rot="R180"/>
-<attribute name="POPULARITY" value="77" x="-15.24" y="-30.48" size="1.778" layer="27" rot="R270" display="off"/>
-<attribute name="SPICEPREFIX" value="R" x="-15.24" y="-30.48" size="1.778" layer="27" rot="R270" display="off"/>
-<attribute name="VALUE" x="34.925" y="26.035" size="0.6096" layer="27" rot="R180"/>
-</element>
 <element name="R11" library="rcl" library_urn="urn:adsk.eagle:library:334" package="R0603" package3d_urn="urn:adsk.eagle:package:23555/3" value="100kΩ" x="20.32" y="19.05" smashed="yes" rot="R180">
 <attribute name="NAME" x="19.685" y="18.415" size="0.6096" layer="25" rot="R180"/>
@@
 <attribute name="POPULARITY" value="40" x="8.89" y="59.69" size="1.778" layer="27" rot="R90" display="off"/>
 <attribute name="VALUE" x="13.97" y="57.15" size="0.6096" layer="27" ratio="10" rot="R90"/>
+</element>
+<element name="R10" library="rcl" library_urn="urn:adsk.eagle:library:334" package="R0603" package3d_urn="urn:adsk.eagle:package:23555/3" value="100Ω" x="35.56" y="26.67" smashed="yes">
+<attribute name="NAME" x="34.925" y="27.305" size="0.6096" layer="25"/>
+<attribute name="POPULARITY" value="77" x="35.56" y="26.67" size="1.778" layer="27" display="off"/>
+<attribute name="SPICEPREFIX" value="R" x="35.56" y="26.67" size="1.778" layer="27" display="off"/>
+<attribute name="VALUE" x="34.925" y="24.765" size="0.6096" layer="27"/>
 </element>
 </elements>
@@
 <contactref element="R30" pad="2"/>
 <contactref element="COMPARATEUR" pad="2"/>
-<contactref element="R10" pad="2"/>
 <contactref element="NMOS" pad="2"/>
 <polygon width="0.1524" layer="1">
@@
 <signal name="N$22">
 <contactref element="COMPARATEUR" pad="1"/>
-<contactref element="NMOS" pad="1"/>
-<contactref element="R10" pad="1"/>
-<wire x1="46.67" y1="21.62" x2="46.67" y2="23.18" width="0.1524" layer="1"/>
-<wire x1="46.67" y1="23.18" x2="45.72" y2="24.13" width="0.1524" layer="1"/>
-<via x="45.72" y="24.13" extent="1-16" drill="0.35"/>
-<wire x1="35.56" y1="28.79" x2="35.98" y2="29.21" width="0.1524" layer="1"/>
-<wire x1="40.64" y1="29.21" x2="42.13" y2="27.72" width="0.1524" layer="1"/>
-<wire x1="42.13" y1="27.72" x2="42.13" y2="27.63" width="0.1524" layer="1"/>
-<wire x1="35.98" y1="29.21" x2="39.37" y2="29.21" width="0.1524" layer="1"/>
-<wire x1="39.37" y1="29.21" x2="40.64" y2="29.21" width="0.1524" layer="1"/>
-<via x="39.37" y="29.21" extent="1-16" drill="0.35"/>
-<wire x1="45.72" y1="24.13" x2="43.18" y2="24.13" width="0.1524" layer="16"/>
-<wire x1="43.18" y1="24.13" x2="39.37" y2="27.94" width="0.1524" layer="16"/>
-<wire x1="39.37" y1="27.94" x2="39.37" y2="29.21" width="0.1524" layer="16"/>
+<contactref element="R10" pad="2"/>
+<wire x1="46.67" y1="21.62" x2="46.67" y2="23.561" width="0.1524" layer="1"/>
+<wire x1="36.41" y1="25.312" x2="36.41" y2="26.67" width="0.1524" layer="1"/>
+<wire x1="46.67" y1="23.561" x2="45.72" y2="24.511" width="0.1524" layer="1"/>
+<wire x1="45.72" y1="24.511" x2="37.211" y2="24.511" width="0.1524" layer="1"/>
+<wire x1="37.211" y1="24.511" x2="36.41" y2="25.312" width="0.1524" layer="1"/>
 </signal>
 <signal name="N$32">
@@
 <wire x1="12.7" y1="46.99" x2="19.05" y2="46.99" width="0.1524" layer="1"/>
 </signal>
+<signal name="N$33">
+<contactref element="R10" pad="1"/>
+<contactref element="NMOS" pad="1"/>
+<wire x1="34.71" y1="26.67" x2="34.71" y2="27.09" width="0.1524" layer="1"/>
+<wire x1="34.71" y1="27.09" x2="35.56" y2="27.94" width="0.1524" layer="1"/>
+<wire x1="35.56" y1="27.94" x2="41.82" y2="27.94" width="0.1524" layer="1"/>
+<wire x1="41.82" y1="27.94" x2="42.13" y2="27.63" width="0.1524" layer="1"/>
+</signal>
 </signals>
