File: EL_Electrical/Autre/Accumulator indicator voltage/Indicator_voltage_TNN_V1.0.sch (EAGLE design)
At the start: 55 parts, among them J2 22-27-2021

Commit message: Finalisation_carte_élec_V1.0
Parts:
- R10: value 10kΩ, 2W -> 100Ω
Connections:
- new net N$33: NMOS.G, R10.1
- net N$22: now also R10.2; no longer NMOS.G, R10.1
- net V-: no longer R10.2
Other:
- moved on the sheet: R10
Changed lines of the file:
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@@
 <setting verticaltext="up"/>
 </settings>
-<grid distance="0.1" unitdist="inch" unit="inch" style="lines" multiple="1" display="no" altdistance="0.01" altunitdist="inch" altunit="inch"/>
+<grid distance="2.54" unitdist="mm" unit="mm" style="lines" multiple="1" display="yes" altdistance="0.254" altunitdist="mm" altunit="mm"/>
 <layers>
 <layer number="1" name="Top" color="4" fill="1" visible="no" active="no"/>
@@
 <part name="P-7" library="supply1" library_urn="urn:adsk.eagle:library:371" deviceset="V-" device="" value="HV-"/>
 <part name="NMOS" library="DMN2041L-7" deviceset="DMN2041L-7" device="" value="SOT-23"/>
-<part name="R10" library="rcl" library_urn="urn:adsk.eagle:library:334" deviceset="R-US_" device="R0603" package3d_urn="urn:adsk.eagle:package:23555/3" value="10kΩ, 2W"/>
-<part name="P-8" library="supply1" library_urn="urn:adsk.eagle:library:371" deviceset="V-" device="" value="HV-"/>
 <part name="P-9" library="supply1" library_urn="urn:adsk.eagle:library:371" deviceset="V-" device="" value="HV-"/>
 <part name="R9" library="wirepad" library_urn="urn:adsk.eagle:library:412" deviceset="1,6/0,8" device="" package3d_urn="urn:adsk.eagle:package:30830/1" value="100Ω, 2W"/>
@@
 <part name="HV+" library="con-molex" library_urn="urn:adsk.eagle:library:165" deviceset="22-23-2021" device="" package3d_urn="urn:adsk.eagle:package:8078633/1"/>
 <part name="HV-" library="con-molex" library_urn="urn:adsk.eagle:library:165" deviceset="22-23-2021" device="" package3d_urn="urn:adsk.eagle:package:8078633/1"/>
+<part name="R10" library="rcl" library_urn="urn:adsk.eagle:library:334" deviceset="R-US_" device="R0603" package3d_urn="urn:adsk.eagle:package:23555/3" value="100Ω"/>
 </parts>
 <sheets>
@@
 <attribute name="VALUE" x="191.77" y="336.55" size="1.778" layer="96" align="center-left"/>
 </instance>
-<instance part="R10" gate="G$1" x="175.26" y="325.12" smashed="yes" rot="R270">
-<attribute name="NAME" x="179.07" y="326.6186" size="1.778" layer="95"/>
-<attribute name="VALUE" x="179.07" y="324.358" size="1.778" layer="96"/>
-</instance>
-<instance part="P-8" gate="1" x="175.26" y="314.96" smashed="yes">
-<attribute name="VALUE" x="175.26" y="312.42" size="1.778" layer="96" rot="R180"/>
-</instance>
 <instance part="P-9" gate="1" x="187.96" y="314.96" smashed="yes">
 <attribute name="VALUE" x="187.96" y="312.42" size="1.778" layer="96" rot="R180"/>
@@
 </instance>
 <instance part="HV-" gate="-2" x="30.48" y="302.26" smashed="yes"/>
+<instance part="R10" gate="G$1" x="170.18" y="335.28" smashed="yes" rot="R180">
+<attribute name="NAME" x="168.91" y="339.3186" size="1.778" layer="95"/>
+<attribute name="VALUE" x="168.91" y="337.058" size="1.778" layer="96"/>
+</instance>
 </instances>
 <busses>
@@
 <pinref part="COMPARATEUR" gate="G$1" pin="VCC-"/>
 <wire x1="154.94" y1="340.36" x2="154.94" y2="332.74" width="0.1524" layer="91"/>
-</segment>
-<segment>
-<pinref part="R10" gate="G$1" pin="2"/>
-<pinref part="P-8" gate="1" pin="V-"/>
-<wire x1="175.26" y1="320.04" x2="175.26" y2="317.5" width="0.1524" layer="91"/>
 </segment>
 <segment>
@@
 <pinref part="COMPARATEUR" gate="G$1" pin="OUT"/>
 <wire x1="157.48" y1="332.74" x2="157.48" y2="335.28" width="0.1524" layer="91"/>
-<pinref part="NMOS" gate="G$1" pin="G"/>
-<wire x1="157.48" y1="335.28" x2="175.26" y2="335.28" width="0.1524" layer="91"/>
-<pinref part="R10" gate="G$1" pin="1"/>
-<wire x1="175.26" y1="335.28" x2="180.34" y2="335.28" width="0.1524" layer="91"/>
-<wire x1="175.26" y1="335.28" x2="175.26" y2="330.2" width="0.1524" layer="91"/>
-<junction x="175.26" y="335.28"/>
+<pinref part="R10" gate="G$1" pin="2"/>
+<wire x1="165.1" y1="335.28" x2="157.48" y2="335.28" width="0.1524" layer="91"/>
 </segment>
 </net>
@@
 </segment>
 </net>
+<net name="N$33" class="0">
+<segment>
+<pinref part="R10" gate="G$1" pin="1"/>
+<pinref part="NMOS" gate="G$1" pin="G"/>
+<wire x1="175.26" y1="335.28" x2="180.34" y2="335.28" width="0.1524" layer="91"/>
+</segment>
+</net>
