File: EL_Electrical/Autre/Shutdown_circuit/Precharge circuit/Precharge_circuit_logic_TNN_V1.0.brd (EAGLE design)
At the start: 64.8 x 45.7 mm, 51 parts, among them IC1 L4941BDT-TR, IC2 TS391ILT, IC3 ADUM5242ARZ, Q1 DMN2041L-7

Commit message: Finalisation_carte_élec_V1.0
Parts:
- R27, R28: value 10kΩ -> 100Ω
- moved R28 1.09 mm to (35.8, 32.6), turned to 90 degrees
- moved R27 0.95 mm to (30.8, 33.6), turned to 0 degrees
Connections:
- new net N$29: NMOS.1, R28.1
- new net N$30: Q1.1, R27.1
- net GND: no longer R27.1, R28.1
- net N$26: no longer Q1.1
- net N$27: no longer NMOS.1
Routing:
- net GND: track 82.2 -> 76.7 mm
- net N$30: track 0.00 -> 2.54 mm
- net N$26: track 20.2 -> 18.3 mm
- net N$29: track 0.00 -> 1.63 mm
- net N$27: track 10.5 -> 9.09 mm, vias 3 -> 2
Changed lines of the file:
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@@
 <attribute name="VALUE" x="33.655" y="17.78" size="0.6096" layer="27"/>
-</element>
-<element name="R27" library="rcl" library_urn="urn:adsk.eagle:library:334" package="R0603" package3d_urn="urn:adsk.eagle:package:23555/3" value="10kΩ" x="31.75" y="33.655" smashed="yes" rot="R180">
-<attribute name="NAME" x="29.845" y="35.56" size="0.6096" layer="25" rot="R180"/>
-<attribute name="POPULARITY" value="77" x="13.97" y="92.075" size="1.778" layer="27" rot="R180" display="off"/>
-<attribute name="SPICEPREFIX" value="R" x="13.97" y="92.075" size="1.778" layer="27" rot="R180" display="off"/>
-<attribute name="VALUE" x="29.845" y="34.29" size="0.6096" layer="27" rot="R180"/>
-</element>
-<element name="R28" library="rcl" library_urn="urn:adsk.eagle:library:334" package="R0603" package3d_urn="urn:adsk.eagle:package:23555/3" value="10kΩ" x="36.83" y="33.02" smashed="yes" rot="R180">
-<attribute name="NAME" x="38.1" y="33.02" size="0.6096" layer="25"/>
-<attribute name="POPULARITY" value="77" x="12.7" y="91.44" size="1.778" layer="27" rot="R180" display="off"/>
-<attribute name="SPICEPREFIX" value="R" x="12.7" y="91.44" size="1.778" layer="27" rot="R180" display="off"/>
-<attribute name="VALUE" x="38.1" y="31.75" size="0.6096" layer="27"/>
 </element>
 <element name="R3" library="rcl" library_urn="urn:adsk.eagle:library:334" package="R0603" package3d_urn="urn:adsk.eagle:package:23555/3" value="100kΩ" x="13.97" y="6.35" smashed="yes" grouprefs="Z">
@@
 <attribute name="OC_NEWARK" value="38C0355" x="60.96" y="30.48" size="1.778" layer="27" rot="R270" display="off"/>
 <attribute name="POPULARITY" value="21" x="60.96" y="30.48" size="1.778" layer="27" rot="R270" display="off"/>
+</element>
+<element name="R27" library="rcl" library_urn="urn:adsk.eagle:library:334" package="R0603" package3d_urn="urn:adsk.eagle:package:23555/3" value="100Ω" x="30.7975" y="33.5915" smashed="yes">
+<attribute name="NAME" x="30.1625" y="34.2265" size="0.6096" layer="25"/>
+<attribute name="POPULARITY" value="77" x="30.7975" y="33.5915" size="1.778" layer="27" display="off"/>
+<attribute name="SPICEPREFIX" value="R" x="30.7975" y="33.5915" size="1.778" layer="27" display="off"/>
+<attribute name="VALUE" x="30.1625" y="31.6865" size="0.6096" layer="27"/>
+</element>
+<element name="R28" library="rcl" library_urn="urn:adsk.eagle:library:334" package="R0603" package3d_urn="urn:adsk.eagle:package:23555/3" value="100Ω" x="35.814" y="32.639" smashed="yes" rot="R90">
+<attribute name="NAME" x="35.179" y="32.004" size="0.6096" layer="25" rot="R90"/>
+<attribute name="POPULARITY" value="77" x="35.814" y="32.639" size="1.778" layer="27" rot="R90" display="off"/>
+<attribute name="SPICEPREFIX" value="R" x="35.814" y="32.639" size="1.778" layer="27" rot="R90" display="off"/>
+<attribute name="VALUE" x="37.719" y="32.004" size="0.6096" layer="27" rot="R90"/>
 </element>
 </elements>
@@
 <contactref element="R25" pad="2"/>
 <contactref element="C5" pad="2"/>
-<contactref element="R27" pad="1"/>
-<contactref element="R28" pad="1"/>
 <contactref element="NMOS" pad="2"/>
 <contactref element="Q1" pad="2"/>
@@
 <wire x1="31.115" y1="11.975" x2="33.11" y2="13.97" width="0.1524" layer="1"/>
 <wire x1="32.71" y1="35.78" x2="32.71" y2="33.765" width="0.1524" layer="1"/>
-<wire x1="32.71" y1="33.765" x2="32.6" y2="33.655" width="0.1524" layer="1"/>
 <wire x1="33.02" y1="31.33" x2="32.71" y2="31.64" width="0.1524" layer="1"/>
 <wire x1="32.71" y1="31.64" x2="32.71" y2="33.765" width="0.1524" layer="1"/>
 <wire x1="33.02" y1="31.33" x2="33.655" y2="31.33" width="0.1524" layer="1"/>
-<wire x1="33.655" y1="31.33" x2="37.045" y2="31.33" width="0.1524" layer="1"/>
-<wire x1="37.68" y1="31.965" x2="37.68" y2="33.02" width="0.1524" layer="1"/>
-<wire x1="37.045" y1="31.33" x2="37.68" y2="31.965" width="0.1524" layer="1"/>
 <wire x1="35.78" y1="28.25" x2="35.455" y2="28.575" width="0.1524" layer="1"/>
 <wire x1="35.455" y1="28.575" x2="34.925" y2="28.575" width="0.1524" layer="1"/>
@@
 <contactref element="R24" pad="1"/>
 <contactref element="IC3" pad="2"/>
-<contactref element="Q1" pad="1"/>
-<contactref element="R27" pad="2"/>
 <wire x1="25.3238" y1="21.59" x2="29.845" y2="21.59" width="0.1524" layer="1"/>
 <via x="29.845" y="21.59" extent="1-16" drill="0.35"/>
@@
 <wire x1="30.48" y1="22.225" x2="30.48" y2="32.385" width="0.1524" layer="16"/>
 <via x="30.48" y="32.385" extent="1-16" drill="0.35"/>
-<wire x1="30.48" y1="32.385" x2="30.9" y2="32.805" width="0.1524" layer="1"/>
-<wire x1="30.9" y1="32.805" x2="30.9" y2="33.655" width="0.1524" layer="1"/>
 <wire x1="30.48" y1="32.385" x2="30.48" y2="31.33" width="0.1524" layer="1"/>
-<wire x1="30.9" y1="33.655" x2="30.9" y2="35.67" width="0.1524" layer="1"/>
-<wire x1="30.9" y1="35.67" x2="30.79" y2="35.78" width="0.1524" layer="1"/>
+<contactref element="R27" pad="2"/>
+<wire x1="31.6475" y1="33.5915" x2="30.48" y2="32.424" width="0.1524" layer="1"/>
+<wire x1="30.48" y1="32.424" x2="30.48" y2="32.385" width="0.1524" layer="1"/>
 </signal>
 <signal name="N$12">
@@
 </signal>
 <signal name="N$27">
-<contactref element="NMOS" pad="1"/>
 <contactref element="COMPARATEUR" pad="1"/>
 <contactref element="R28" pad="2"/>
-<wire x1="32.7" y1="26.7" x2="33.625" y2="26.7" width="0.1524" layer="1"/>
-<wire x1="33.625" y1="26.7" x2="33.655" y2="26.67" width="0.1524" layer="1"/>
-<wire x1="33.655" y1="26.67" x2="34.29" y2="27.305" width="0.1524" layer="1"/>
-<via x="34.29" y="27.305" extent="1-16" drill="0.35"/>
-<wire x1="34.29" y1="27.305" x2="35.56" y2="28.575" width="0.1524" layer="16"/>
-<wire x1="35.56" y1="28.575" x2="35.56" y2="29.21" width="0.1524" layer="16"/>
-<wire x1="35.56" y1="29.21" x2="35.56" y2="31.75" width="0.1524" layer="16"/>
-<wire x1="35.56" y1="31.75" x2="34.925" y2="32.385" width="0.1524" layer="16"/>
-<wire x1="34.925" y1="32.385" x2="34.925" y2="33.02" width="0.1524" layer="16"/>
-<via x="34.925" y="33.02" extent="1-16" drill="0.35"/>
-<wire x1="34.925" y1="33.02" x2="35.98" y2="33.02" width="0.1524" layer="1"/>
-<wire x1="35.78" y1="30.17" x2="35.78" y2="29.43" width="0.1524" layer="1"/>
-<wire x1="35.78" y1="29.43" x2="35.56" y2="29.21" width="0.1524" layer="1"/>
-<via x="35.56" y="29.21" extent="1-16" drill="0.35"/>
+<wire x1="32.7" y1="26.7" x2="33.6215" y2="26.7" width="0.1524" layer="1"/>
+<wire x1="33.6215" y1="26.7" x2="34.29" y2="27.3685" width="0.1524" layer="1"/>
+<via x="34.29" y="27.3685" extent="1-16" drill="0.35"/>
+<wire x1="34.29" y1="27.3685" x2="34.29" y2="32.766" width="0.1524" layer="16"/>
+<via x="34.29" y="32.766" extent="1-16" drill="0.35"/>
+<wire x1="34.29" y1="32.766" x2="35.013" y2="33.489" width="0.1524" layer="1"/>
+<wire x1="35.013" y1="33.489" x2="35.814" y2="33.489" width="0.1524" layer="1"/>
 </signal>
 <signal name="N$28">
@@
 <wire x1="58.42" y1="14.605" x2="58.42" y2="16.51" width="0.508" layer="1"/>
 </signal>
+<signal name="N$29">
+<contactref element="R28" pad="1"/>
+<contactref element="NMOS" pad="1"/>
+<wire x1="35.814" y1="31.789" x2="35.78" y2="31.755" width="0.1524" layer="1"/>
+<wire x1="35.78" y1="31.755" x2="35.78" y2="30.17" width="0.1524" layer="1"/>
+</signal>
+<signal name="N$30">
+<contactref element="R27" pad="1"/>
+<contactref element="Q1" pad="1"/>
+<wire x1="30.79" y1="35.78" x2="29.9475" y2="34.9375" width="0.1524" layer="1"/>
+<wire x1="29.9475" y1="34.9375" x2="29.9475" y2="33.5915" width="0.1524" layer="1"/>
+</signal>
 </signals>
