File: EL_Electrical/Autre/TSAL/TSAL_contactor_state_and_accumulator_voltage_measurement/TSAL_contactor_state_and_accumulator_voltage_measurement_TNN_V1.0.brd (EAGLE design)
At the start: 48.3 x 24.1 mm, 30 parts, among them IC2 L4941BDT-TR, IC5 TS391ILT, IC6 ADUM5242ARZ

Commit message: Finalisation_carte_élec_V1.0
Parts:
- removed R14: 10kΩ, rcl:R0603
Connections:
- net +5V_ISO: no longer R14.1
- net VOLTAGE_ON_ACCUMULATOR_ISO: no longer R14.2
Routing:
- net +5V_ISO: track 24.2 -> 18.2 mm, vias 3 -> 2
- net VOLTAGE_ON_ACCUMULATOR_ISO: track 11.1 -> 10.5 mm
Changed lines of the file:
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@@
 <attribute name="VALUE" x="7.874" y="4.826" size="0.6096" layer="27" rot="R180"/>
-</element>
-<element name="R14" library="rcl" library_urn="urn:adsk.eagle:library:334" package="R0603" package3d_urn="urn:adsk.eagle:package:23555/3" value="10kΩ" x="10.287" y="10.414" smashed="yes" rot="R270">
-<attribute name="NAME" x="9.652" y="11.43" size="0.6096" layer="25" rot="R180"/>
-<attribute name="POPULARITY" value="77" x="-34.163" y="-40.386" size="1.778" layer="27" rot="R270" display="off"/>
-<attribute name="SPICEPREFIX" value="R" x="-34.163" y="-40.386" size="1.778" layer="27" rot="R270" display="off"/>
-<attribute name="VALUE" x="9.652" y="10.795" size="0.6096" layer="27" rot="R180"/>
 </element>
 <element name="R15" library="rcl" library_urn="urn:adsk.eagle:library:334" package="R0603" package3d_urn="urn:adsk.eagle:package:23555/3" value="10kΩ" x="40.64" y="12.192" smashed="yes">
@@
 <contactref element="C5" pad="2"/>
 <contactref element="R13" pad="2"/>
-<contactref element="R14" pad="1"/>
 <contactref element="IC6" pad="8"/>
 <wire x1="13.238" y1="8.062" x2="13.208" y2="8.062" width="0.1524" layer="1"/>
@@
 <wire x1="7.874" y1="7.366" x2="11.938" y2="7.366" width="0.1524" layer="16"/>
 <via x="11.938" y="7.366" extent="1-16" drill="0.35"/>
-<wire x1="10.287" y1="11.264" x2="8.47" y2="11.264" width="0.1524" layer="1"/>
-<wire x1="8.47" y1="11.264" x2="7.874" y2="10.668" width="0.1524" layer="1"/>
-<via x="7.874" y="10.668" extent="1-16" drill="0.35"/>
-<wire x1="7.874" y1="10.668" x2="7.874" y2="7.366" width="0.1524" layer="16"/>
 <wire x1="17.8562" y1="10.795" x2="14.097" y2="10.795" width="0.1524" layer="1"/>
 <wire x1="14.097" y1="10.795" x2="13.716" y2="10.414" width="0.1524" layer="1"/>
@@
 <signal name="VOLTAGE_ON_ACCUMULATOR_ISO">
 <contactref element="IC5" pad="1"/>
-<contactref element="R14" pad="2"/>
 <contactref element="IC6" pad="7"/>
 <wire x1="17.8562" y1="12.065" x2="11.811" y2="12.065" width="0.1524" layer="1"/>
 <wire x1="11.811" y1="12.065" x2="11.176" y2="11.43" width="0.1524" layer="1"/>
-<wire x1="11.176" y1="11.43" x2="11.176" y2="9.906" width="0.1524" layer="1"/>
-<wire x1="11.176" y1="9.906" x2="10.834" y2="9.564" width="0.1524" layer="1"/>
-<wire x1="10.834" y1="9.564" x2="10.287" y2="9.564" width="0.1524" layer="1"/>
-<wire x1="10.287" y1="9.564" x2="10.638" y2="9.213" width="0.1524" layer="1"/>
-<wire x1="10.638" y1="9.213" x2="10.638" y2="8.062" width="0.1524" layer="1"/>
+<wire x1="11.176" y1="9.906" x2="11.176" y2="11.43" width="0.1524" layer="1"/>
+<wire x1="10.638" y1="9.213" x2="10.638" y2="8.89" width="0.1524" layer="1"/>
+<wire x1="10.638" y1="8.89" x2="10.638" y2="8.062" width="0.1524" layer="1"/>
+<wire x1="10.638" y1="9.213" x2="10.638" y2="9.368" width="0.1524" layer="1"/>
+<wire x1="10.638" y1="9.368" x2="11.176" y2="9.906" width="0.1524" layer="1"/>
 </signal>
 </signals>
