File: EL_Electrical/Autre/TSAL/TSAL_inverter_voltage_measurement/TSAL_inverter_voltage_measurement_TNN_V1.0.sch (EAGLE design)
At the start: 26 parts, among them IC1 L4941BDT-TR, IC2 TS391ILT, IC3 ADUM5242ARZ

Commit message: Finalisation_carte_élec_V1.0
Parts:
- removed R13: 10kΩ, rcl:R-US_R0603
Connections:
- net +5V_ISO: no longer R13.1
- net VOLTAGE_ON_INVERTER_ISO: no longer R13.2
Changed lines of the file:
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@@
 <setting verticaltext="up"/>
 </settings>
-<grid distance="0.1" unitdist="inch" unit="mm" style="lines" multiple="1" display="yes" altdistance="0.01" altunitdist="inch" altunit="mm"/>
+<grid distance="2.54" unitdist="mm" unit="mm" style="lines" multiple="1" display="yes" altdistance="0.254" altunitdist="mm" altunit="mm"/>
 <layers>
 <layer number="1" name="Top" color="4" fill="1" visible="no" active="no"/>
@@
 <part name="R12" library="rcl" library_urn="urn:adsk.eagle:library:334" deviceset="R-US_" device="R0603" package3d_urn="urn:adsk.eagle:package:23555/3" value="100kΩ"/>
 <part name="IC3" library="ADUM5242ARZ" deviceset="ADUM5242ARZ" device=""/>
-<part name="R13" library="rcl" library_urn="urn:adsk.eagle:library:334" deviceset="R-US_" device="R0603" package3d_urn="urn:adsk.eagle:package:23555/3" value="10kΩ"/>
 <part name="GND3" library="supply1" library_urn="urn:adsk.eagle:library:371" deviceset="GND" device=""/>
 <part name="P+4" library="supply1" library_urn="urn:adsk.eagle:library:371" deviceset="+5V" device=""/>
@@
 <attribute name="VALUE" x="87.63" y="106.68" size="1.778" layer="96" align="center-left"/>
 </instance>
-<instance part="R13" gate="G$1" x="139.7" y="162.56" smashed="yes">
-<attribute name="NAME" x="135.89" y="166.5986" size="1.778" layer="95"/>
-<attribute name="VALUE" x="135.89" y="164.338" size="1.778" layer="96"/>
-</instance>
 <instance part="GND3" gate="1" x="76.2" y="88.9" smashed="yes">
 <attribute name="VALUE" x="73.66" y="91.44" size="1.778" layer="96" rot="R180"/>
@@
 </segment>
 <segment>
-<pinref part="R13" gate="G$1" pin="1"/>
-<wire x1="134.62" y1="162.56" x2="129.54" y2="162.56" width="0.1524" layer="91"/>
-<label x="129.54" y="162.56" size="1.778" layer="95" rot="R180" xref="yes"/>
-</segment>
-<segment>
 <pinref part="IC3" gate="G$1" pin="VISO"/>
 <wire x1="109.22" y1="101.6" x2="111.76" y2="101.6" width="0.1524" layer="91"/>
@@
 <wire x1="147.32" y1="162.56" x2="149.86" y2="162.56" width="0.1524" layer="91"/>
 <label x="149.86" y="162.56" size="1.778" layer="95" xref="yes"/>
-<pinref part="R13" gate="G$1" pin="2"/>
-<wire x1="147.32" y1="162.56" x2="144.78" y2="162.56" width="0.1524" layer="91"/>
-<junction x="147.32" y="162.56"/>
-</segment>
-<segment>
+</segment>
+<segment>
